File: electronics/trezor_v1.1_usb_c/trezor_v1.1.kicad_sch (KiCad schematic)
At the start: 34 parts

Commit message: cleanup: fix 3d models in pcb
Parts:
- C1, C18, C2, C3, C4: value (none) -> 1u; footprint (none) -> trezor_v1.1:0402
- C10: value (none) -> 4u7; footprint (none) -> trezor_v1.1:0603
- C12, C13, C14, C15, C16, C7, C9: value (none) -> 100n; footprint (none) -> trezor_v1.1:0402
- C20, C21: value (none) -> 22p; footprint (none) -> trezor_v1.1:0402
- C5: value (none) -> 2u2; footprint (none) -> trezor_v1.1:0603
- C6, C8: value (none) -> 2u2; footprint (none) -> trezor_v1.1:0402
- D2: value (none) -> BAT60BWS; footprint (none) -> trezor_v1.1:SOD323
- IC1: value (none) -> MCP1703T-3302E/CB; footprint (none) -> trezor_v1.1:SOT23
- J1: value (none) -> USB_C_Receptacle_USB2.0
- K2: value (none) -> SWD; footprint (none) -> trezor_v1.1:SWD
- Q2: value (none) -> 8MHz; footprint (none) -> trezor_v1.1:CTS406
- R1, R5: value (none) -> 5.1k; footprint (none) -> trezor_v1.1:0402
- R10: value (none) -> 390k; footprint (none) -> trezor_v1.1:0402
- R2: value (none) -> MF-FSMF020X-2; footprint (none) -> trezor_v1.1:0603
- R3, R4: value (none) -> 22R; footprint (none) -> trezor_v1.1:0402
- R7: value (none) -> 12k; footprint (none) -> trezor_v1.1:0402
- S1, S2: value (none) -> SWITCH-MOMENTARY-2SMD; footprint (none) -> trezor_v1.1:TACTILE_SWITCH_SMD
- U1: value (none) -> STM32F205RET6; footprint (none) -> trezor_v1.1:TQFP64
- U3: value (none) -> DISPLAY; footprint (none) -> trezor_v1.1:UG-2864HSWEG01_0.96IN_WRAPAROUND

Commit message: cleanup: cleanup silkscreen, add revision info
Parts:
- J1: footprint (none) -> Gigahawk:USB_C_Receptacle_GCT_USB4085
Connections:
- no-connect marks 2 -> 31
Other:
- title: (none) -> Trezor One USB-C
- moved on the sheet: C1, C10, C12, C13, C14, C16, C18, C2, C3, C4, C5, C7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
